File: PODdrive.sch (KiCad schematic (older format))
At the start: 46 parts

Commit message: 160503
rework
Parts:
- removed D?: LED, ~, symbol LED-RESCUE-PODdrive
- removed P?: CONN_1, symbol CONN_1
- removed P? (x2): CONN_8X2, symbol CONN_8X2
- removed R?: R, ~, symbol R-RESCUE-PODdrive
- removed U?: PCF8574, symbol PCF8574-RESCUE-PODdrive
- added D?: LED, ~, symbol LED-RESCUE-PODdrive
- added JP?: JUMPER, symbol JUMPER
- added P?: CONN_ESC1, symbol CONN_01X03
- added P?: CONN_ESC2, symbol CONN_01X03
- added P?: CONN_ESC3, symbol CONN_01X03
- added P?: CONN_ESC4, symbol CONN_01X03
- added P?: CONN_STEPPER1, symbol CONN_01X04
- added P?: CONN_STEPPER2, symbol CONN_01X04
- added P?: CONN_STEPPER3, symbol CONN_01X04
- added P?: CONN_STEPPER4, symbol CONN_01X04
- added P?: CONN_ISP1, symbol CONN_01X06
- added P?: CONN_ISP2, symbol CONN_01X06
- added P?: CONN_01X03_RC_IN, symbol CONN_01X03
- added P? (x2): CONN_8X2, symbol CONN_8X2
- added R?: R, ~, symbol R-RESCUE-PODdrive
- added U?: PCF8574, symbol PCF8574-RESCUE-PODdrive
Connections:
- net labels added: Button_Enter, Button_Left, Button_Right, DO1, DO10, DO11, DO12, DO13, DO14, DO15, DO16, DO2, DO3, DO4, DO5, DO6, DO7, DO8, DO9, GND-RESCUE-PODdrive, HALL1, HALL2, HALL3, HALL4, I2C_SCL, I2C_SDA, LED_1, LED_2, LED_3, LED_4, MISO1, MOSI1, RC_IN, RESET, SCK1, SRV_CH1, SRV_CH2, SRV_CH3, SRV_CH4
- wire segments 237 -> 180
Other:
- moved on the sheet: D?, K?, P?, R?, SW?, U?

Commit message: 160503
capasitors
Parts:
- added C? (x4): CP, symbol CP
Changed lines of the file:
@@
+	1    0    0    -1
+$EndComp
+$Comp
+L CP C?
+U 1 1 5728BC66
+P 2150 10350
+F 0 "C?" H 2175 10450 50  0000 L CNN
+F 1 "CP" H 2175 10250 50  0000 L CNN
+F 2 "" H 2188 10200 50  0000 C CNN
+F 3 "" H 2150 10350 50  0000 C CNN
+	1    2150 10350
+	1    0    0    -1
+$EndComp
+$Comp
+L CP C?
+U 1 1 5728BDAB
+P 3300 10350
+F 0 "C?" H 3325 10450 50  0000 L CNN
+F 1 "CP" H 3325 10250 50  0000 L CNN
+F 2 "" H 3338 10200 50  0000 C CNN
+F 3 "" H 3300 10350 50  0000 C CNN
+	1    3300 10350
+	1    0    0    -1
+$EndComp
+$Comp
+L CP C?
+U 1 1 5728BEEC
+P 4400 10300
+F 0 "C?" H 4425 10400 50  0000 L CNN
+F 1 "CP" H 4425 10200 50  0000 L CNN
+F 2 "" H 4438 10150 50  0000 C CNN
+F 3 "" H 4400 10300 50  0000 C CNN
+	1    4400 10300
+	1    0    0    -1
+$EndComp
+$Comp
+L CP C?
+U 1 1 5728C04A
+P 5350 10300
+F 0 "C?" H 5375 10400 50  0000 L CNN
+F 1 "CP" H 5375 10200 50  0000 L CNN
+F 2 "" H 5388 10150 50  0000 C CNN
+F 3 "" H 5350 10300 50  0000 C CNN
+	1    5350 10300
 	1    0    0    -1
 $EndComp

Commit message: 160503
update i2c
Parts:
- removed P? (x2): CONN_3X2, symbol CONN_3X2
- added P?: CONN_LCD, symbol CONN_01X04
Connections:
- net I2C_SCL: now also IC?.22 ((PCINT16/SCL)PC0), R?.2
- net I2C_SDA: now also IC?.23 ((PCINT17/SDA)PC1), R?.2
- net LED_4: no longer IC?.18 ((PCINT6/MISO/DO)PB6)
- now unconnected: IC?.17 ((PCINT5/MOSI/DI/SDA)PB5), IC?.19 ((PCINT7/USCK/SCK/SCL)PB7)
Other:
- moved on the sheet: R?

Commit message: added power conn
Parts:
- added P?: CONN_Power, symbol CONN_01X03
Connections:
- net +5V: now also P?.2 (P2)
- net GND: now also P?.3 (P3)
Other:
- moved on the sheet: P?
Changed lines of the file:
@@
 L CONN_01X03 P?
 U 1 1 5728E62B
-P 14300 9200
-F 0 "P?" H 14300 9400 50  0000 C CNN
-F 1 "CONN_01X03_RC_IN" V 14400 9200 50  0000 C CNN
-F 2 "" H 14300 9200 50  0000 C CNN
-F 3 "" H 14300 9200 50  0000 C CNN
-	1    14300 9200
+P 14000 9200
+F 0 "P?" H 14000 9400 50  0000 C CNN
+F 1 "CONN_01X03_RC_IN" V 14100 9200 50  0000 C CNN
+F 2 "" H 14000 9200 50  0000 C CNN
+F 3 "" H 14000 9200 50  0000 C CNN
+	1    14000 9200
 	0    1    1    0
 $EndComp
-Text GLabel 14400 8800 1    60   Input ~ 0
+Text GLabel 14100 8800 1    60   Input ~ 0
 RC_IN
 $Comp
 L +5V #PWR?
 U 1 1 5728F0D2
-P 14300 9000
-F 0 "#PWR?" H 14300 8850 50  0001 C CNN
-F 1 "+5V" H 14300 9140 50  0000 C CNN
-F 2 "" H 14300 9000 50  0000 C CNN
-F 3 "" H 14300 9000 50  0000 C CNN
-	1    14300 9000
+P 14000 9000
+F 0 "#PWR?" H 14000 8850 50  0001 C CNN
+F 1 "+5V" H 14000 9140 50  0000 C CNN
+F 2 "" H 14000 9000 50  0000 C CNN
+F 3 "" H 14000 9000 50  0000 C CNN
+	1    14000 9000
 	1    0    0    -1
 $EndComp
@@
 L GND-RESCUE-PODdrive #PWR?
 U 1 1 5728F696
-P 14200 9000
-F 0 "#PWR?" H 14200 9000 30  0001 C CNN
-F 1 "GND-RESCUE-PODdrive" H 14200 8930 30  0001 C CNN
-F 2 "" H 14200 9000 60  0000 C CNN
-F 3 "" H 14200 9000 60  0000 C CNN
-	1    14200 9000
+P 13900 9000
+F 0 "#PWR?" H 13900 9000 30  0001 C CNN
+F 1 "GND-RESCUE-PODdrive" H 13900 8930 30  0001 C CNN
+F 2 "" H 13900 9000 60  0000 C CNN
+F 3 "" H 13900 9000 60  0000 C CNN
+	1    13900 9000
 	-1   0    0    1
 $EndComp
@@
 Connection ~ 11000 10350
 Wire Wire Line
-	14400 8800 14400 9000
+	14100 8800 14100 9000
 Wire Wire Line
 	4350 3450 4150 3450
@@
 Text GLabel 12200 6700 1    60   BiDi ~ 0
 I2C_SDA
+$Comp
+L CONN_01X03 P?
+U 1 1 5729C8D1
+P 14800 9200
+F 0 "P?" H 14800 9400 50  0000 C CNN
+F 1 "CONN_Power" V 14900 9200 50  0000 C CNN
+F 2 "" H 14800 9200 50  0000 C CNN
+F 3 "" H 14800 9200 50  0000 C CNN
+	1    14800 9200
+	0    1    1    0
+$EndComp
+$Comp
+L GND-RESCUE-PODdrive #PWR?
+U 1 1 5729CB59
+P 14700 9000
+F 0 "#PWR?" H 14700 9000 30  0001 C CNN
+F 1 "GND-RESCUE-PODdrive" H 14700 8930 30  0001 C CNN
+F 2 "" H 14700 9000 60  0000 C CNN
+F 3 "" H 14700 9000 60  0000 C CNN
+	1    14700 9000
+	-1   0    0    1
+$EndComp
+$Comp
+L +5V #PWR?
+U 1 1 5729CC24
+P 14800 9000
+F 0 "#PWR?" H 14800 8850 50  0001 C CNN
+F 1 "+5V" H 14800 9140 50  0000 C CNN
+F 2 "" H 14800 9000 50  0000 C CNN
+F 3 "" H 14800 9000 50  0000 C CNN
+	1    14800 9000
+	1    0    0    -1
+$EndComp
 $EndSCHEMATC

Commit message: optimisation
Parts:
- removed P?: CONN_12, symbol CONN_12
- added P?: CONN_SRV_OUT, symbol CONN_01X12
- added P?: CONN_SRV_SUPPLY, symbol CONN_02X12
Connections:
- net +5V: now also P?.1 (P1), P?.11 (P11), P?.13 (P13), P?.15 (P15), P?.17 (P17), P?.19 (P19), P?.21 (P21), P?.23 (P23), P?.3 (P3), P?.5 (P5), P?.7 (P7), P?.9 (P9)
- net GND: now also C?.2, IC?.1 (PA2(~RESET~/dW)), IC?.9 (~RESET), P?.10 (P10), P?.12 (P12), P?.14 (P14), P?.16 (P16), P?.18 (P18), P?.2 (P2), P?.20 (P20), P?.22 (P22), P?.24 (P24), P?.4 (P4), P?.6 (P6), P?.8 (P8); no longer C?.1
- net I2C_SCL: now also IC?.19 ((PCINT7/USCK/SCK/SCL)PB7)
- net I2C_SDA: now also IC?.17 ((PCINT5/MOSI/DI/SDA)PB5)
- net LED_4: now also IC?.18 ((PCINT6/MISO/DO)PB6)
- net at R?.2: now also SW?.2; no longer SW?.1
- new net: C?.1, SW?.1
Other:
- moved on the sheet: C?, D?, K?, P?, R?, SW?

Commit message: PORT Key LED
Parts:
- P?: value CONN_8X2 -> CONN_DO1-8
- P?: value CONN_8X2 -> CONN_DO9-16
Connections:
- net +5V: now also U?.1 (A0)
- net Button_Enter: now also IC?.6 ((PCINT13/MOSI)PB5)
- net Button_Left: now also IC?.5 ((PCINT12/OC0B/~SS~)PB4)
- net Button_Right: now also IC?.4 ((PCINT11/AIN1/OC0)PB3)
- net DO1: now also P?.1, U?.4 (P0)
- net DO10: now also P?.3, U?.5 (P1)
- net DO11: now also P?.5, U?.6 (P2)
- net DO12: now also P?.7, U?.7 (P3)
- net DO13: now also P?.9, U?.9 (P4)
- net DO14: now also P?.11, U?.10 (P5)
- net DO15: now also P?.13, U?.11 (P6)
- net DO16: now also P?.15, U?.12 (P7)
- net DO2: now also P?.3, U?.5 (P1)
- net DO3: now also P?.5, U?.6 (P2)
- net DO4: now also P?.7, U?.7 (P3)
- net DO5: now also P?.9, U?.9 (P4)
- net DO6: now also P?.11, U?.10 (P5)
- net DO7: now also P?.13, U?.11 (P6)
- net DO8: now also P?.15, U?.12 (P7)
- net DO9: now also P?.1, U?.4 (P0)
- net GND: no longer U?.1 (A0)
- net I2C_SCL: now also U?.14 (SCL), U?.14 (SCL)
- net I2C_SDA: now also U?.15 (SDA), U?.15 (SDA)
- net LED_1: now also IC?.1 ((PCINT8/T0/XCK)PB0)
- net LED_2: now also IC?.2 ((PCINT9/CLKO/T1)PB1)
- net LED_3: now also IC?.3 ((PCINT10/AIN0/INT2)PB2)
- net SRV_CH1: now also IC?.12 ((PCINT0/AIN0)PB0), P?.1 (P1)
- net SRV_CH10: now also IC?.8 ((T0)PD4)
- net SRV_CH11: now also IC?.9 ((OC0B/T1)PD5)
- net SRV_CH12: now also IC?.11 ((ICP)PD6)
- net SRV_CH2: now also IC?.13 ((PCINT1/AIN1)PB1)
- net SRV_CH3: now also IC?.14 ((PCINT2/OC0A)PB2)
- net SRV_CH4: now also IC?.15 ((PCINT3/OC1A)PB3)
- net SRV_CH5: now also IC?.16 ((PCINT4/OC1B)PB4)
- net SRV_CH6: now also IC?.2 ((RXD)PD0)
- net SRV_CH7: now also IC?.3 ((TXD)PD1)
- net SRV_CH8: now also IC?.6 ((CKOUT/XCK/INT0)PD2)
- net SRV_CH9: now also IC?.7 ((INT1)PD3)
- net at P?.6 (P6): now also P?.1 (P1)
- net at P?.7 (P7): now also C?.2, P?.3 (P3)
- net at P?.8 (P8): now also C?.1, P?.2 (P2)
- no-connect marks 0 -> 12
Other:
- moved on the sheet: C?, P?

Commit message: finished
now to be checked
Parts:
- removed C? (x3): CP, symbol CP
- removed K? (x4): CONN_3, symbol CONN_3
- removed P? (x8): CONN_8, symbol CONN_8
- removed P?: CONN_ESC1, symbol CONN_01X03
- removed P?: CONN_ESC2, symbol CONN_01X03
- removed P?: CONN_ESC3, symbol CONN_01X03
- removed P?: CONN_STEPPER1, symbol CONN_01X04
- removed P?: CONN_STEPPER2, symbol CONN_01X04
- removed P?: CONN_STEPPER3, symbol CONN_01X04
- added C? (x3): CP, symbol CP
- added P?: CONN_SPEAKER, symbol CONN_01X02
- added P?: CONN_ESC3, symbol CONN_01X03
- added P?: CONN_STEPPER3, symbol CONN_01X04
- added P?: CONN_ESC2, symbol CONN_01X03
- added P?: CONN_STEPPER2, symbol CONN_01X04
- added P?: CONN_ESC1, symbol CONN_01X03
- added P?: CONN_STEPPER1, symbol CONN_01X04
- added P?: CONN_HALL1, symbol CONN_01X03
- added P?: CONN_HALL2, symbol CONN_01X03
- added P?: CONN_HALL3, symbol CONN_01X03
- added P?: CONN_HALL4, symbol CONN_01X03
- added P?: CONN_UART2, symbol CONN_01X04
- added P?: CONN_UART1, symbol CONN_01X04
- added P?: CONN_ADC, symbol CONN_01X04
- added U? (x4): POLOLU_DRV8433, symbol POLOLU_DRV8433
- added U?: DFPlayer_mini, symbol DFPlayer_mini
Connections:
- net STEP2_STEP is gone; now on net Button_Enter: IC?.35 ((PCINT5/ADC5)PA5)
- net +5V: now also P?.2 (P2), P?.2 (P2), P?.3 (P3), P?.1 (P1), P?.1 (P1), P?.3 (P3), P?.3 (P3), P?.3 (P3), P?.3 (P3), U?.1 (VCC), U?.6 (SLEEP), U?.6 (SLEEP), U?.6 (SLEEP), U?.6 (SLEEP)
- net Button_Enter: no longer IC?.6 ((PCINT13/MOSI)PB5)
- net Button_Left: now also IC?.36 ((PCINT4/ADC4)PA4); no longer IC?.5 ((PCINT12/OC0B/~SS~)PB4)
- net Button_Right: now also IC?.37 ((PCINT3/ADC3)PA3); no longer IC?.4 ((PCINT11/AIN1/OC0)PB3)
- net GND: now also P?.1 (P1), P?.1 (P1), P?.3 (P3), P?.3 (P3), P?.4 (P4), P?.2 (P2), P?.2 (P2), P?.2 (P2), P?.2 (P2), P?.2 (P2), P?.2 (P2), P?.3 (P3), U?.10 (GND), U?.7 (GND), U?.9 (GND), U?.9 (GND), U?.9 (GND), U?.9 (GND)
- net HALL1: now also P?.1 (P1)
- net HALL2: now also P?.1 (P1)
- net HALL3: now also P?.1 (P1)
- net HALL4: now also P?.1 (P1)
- net I2C_SCL: now also P?.1 (P1), P?.4 (P4)
- net I2C_SDA: now also P?.2 (P2), P?.6 (P6)
- net LED_1: now also IC?.40 ((PCINT0/ADC0)PA0); no longer IC?.1 ((PCINT8/T0/XCK)PB0)
- net LED_2: now also IC?.39 ((PCINT1/ADC1)PA1); no longer IC?.2 ((PCINT9/CLKO/T1)PB1)
- net LED_3: now also IC?.38 ((PCINT2/ADC2)PA2); no longer IC?.3 ((PCINT10/AIN0/INT2)PB2)
- net LED_4: now also P?.5 (P5)
- net MISO1: now also IC?.7 ((PCINT14/MISO)PB6), P?.5 (P5), U?.7 (STEP)
- net MOSI1: now also IC?.6 ((PCINT13/MOSI)PB5), P?.6 (P6), U?.7 (STEP)
- net SCK1: now also IC?.8 ((PCINT15/SCK)PB7), P?.4 (P4), U?.7 (STEP)
- net SRV_CH1: now also P?.1 (P1), P?.1 (P1)
- net SRV_CH10: now also P?.10 (P10)
- net SRV_CH11: now also P?.11 (P11)
- net SRV_CH12: now also P?.12 (P12)
- net SRV_CH2: now also P?.2 (P2), P?.1 (P1)
- net SRV_CH3: now also P?.3 (P3), P?.1 (P1)
- net SRV_CH4: now also P?.1 (P1), P?.4 (P4)
- net SRV_CH5: now also P?.5 (P5)
- net SRV_CH6: now also P?.6 (P6)
- net SRV_CH7: now also P?.7 (P7)
- net SRV_CH8: now also P?.8 (P8)
- net SRV_CH9: now also P?.9 (P9)
- net STEP1_DIR: now also IC?.1 ((PCINT8/T0/XCK)PB0), U?.8 (DIR); no longer IC?.40 ((PCINT0/ADC0)PA0)
- net STEP1_STEP: now also IC?.5 ((PCINT12/OC0B/~SS~)PB4), U?.7 (STEP); no longer IC?.36 ((PCINT4/ADC4)PA4)
- net STEP2_DIR: now also IC?.2 ((PCINT9/CLKO/T1)PB1), U?.8 (DIR); no longer IC?.39 ((PCINT1/ADC1)PA1)
- net STEP3_DIR: now also IC?.3 ((PCINT10/AIN0/INT2)PB2), U?.8 (DIR); no longer IC?.38 ((PCINT2/ADC2)PA2)
- net STEP4_DIR: now also IC?.4 ((PCINT11/AIN1/OC0)PB3), U?.8 (DIR); no longer IC?.37 ((PCINT3/ADC3)PA3)
- net RxD0: now reaches IC?.14 ((PCINT24/RXD0)PD0)
- net RxD0: now also P?.3 (P3)
- net TxD0: now reaches IC?.15 ((PCINT25/TXD0)PD1)
- net TxD0: now also P?.4 (P4)
- net RxD1: now reaches IC?.16 ((PCINT26/RXD1/INT0)PD2)
- net RxD1: now also P?.3 (P3), U?.3 (Tx)
- net TxD1: now reaches IC?.17 ((PCINT27/TXD1/INT1)PD3)
- net TxD1: now also P?.4 (P4), U?.2 (Rx)
- net AREF: now reaches IC?.32 (AREF)
- net AREF: now also P?.4 (P4)
- net at P?.2 (P2): now also C?.1, U?.16 (VMOT)
- net at P?.3 (P3): now also C?.2, U?.15 (GND)
- net at P?.1 (P1): now also U?.14 (B2)
- net at P?.2 (P2): now also U?.13 (B1)
- net at P?.3 (P3): now also U?.12 (A1)
- net at P?.4 (P4): now also U?.11 (A2)
- net STEP3_STEP renamed ADC6
- net ADC6: now also P?.1 (P1)
- net STEP4_STEP renamed ADC7
- net ADC7: now also P?.2 (P2)
- new net: P?.2 (P2), U?.6 (SPK_1)
- new net: P?.1 (P1), U?.8 (SPK_2)
- new net: C?.1, P?.2 (P2), U?.16 (VMOT) (x3)
- new net: C?.2, P?.3 (P3), U?.15 (GND) (x3)
- new net: P?.1 (P1), U?.14 (B2) (x3)
- new net: P?.2 (P2), U?.13 (B1) (x3)
- new net: P?.3 (P3), U?.12 (A1) (x3)
- new net: P?.4 (P4), U?.11 (A2) (x3)
- no-connect marks 12 -> 41
Other:
- moved on the sheet: C?, P?, R?
